File: doc/PCB/HALL/HALL.sch (KiCad schematic (older format))
At the start: 92 parts, among them J1 Conn_01x05_Female, J10 CHIN+, J11 CHIN-, J12 Vcc, J13 CHOUT+, J14 CHOUT-, J2 Digit1, J3 Conn_01x05_Female, J4 Digit2, J5 Conn_01x05_Female, J6 Digit3, J7 Conn_01x05_Female, J8 Digit4, J9 PILOT, Q1 BC817-40, Q10 BC817-40, Q11 BC807-40, Q12 BC817-40, Q13 BC817-40, Q14 BC817-40, Q15 IRLR3636, Q16 BC817-40, Q2 BC807-40, Q3 BC817-40, Q4 BC817-40, Q5 BC807-40, Q6 BC817-40, Q7 BC817-40, Q8 BC807-40, Q9 BC817-40, SW1 UP, SW2 LEFT, SW3 RIGHT, SW4 DOWN, SW5 ENTER, SW6 BACK, U1 LM317_3PinPackage, U2 LM7812_TO220, U3 LM1117-3.3, U4 STM32F030K6Tx, U5 LM317_3PinPackage, Y1 Crystal

Commit message: PCB almost done
Parts:
- removed Q1, Q10, Q12, Q13, Q14, Q16, Q3, Q4, Q6, Q7, Q9: BC817-40, Package_TO_SOT_SMD:SOT-23, symbol Transistor_BJT:BC548
- removed Q11, Q2, Q5, Q8: BC807-40, Package_TO_SOT_SMD:SOT-23, symbol Transistor_BJT:BC636
- removed Q15: IRLR3636, Package_TO_SOT_SMD:TO-252-2, symbol Device:Q_NMOS_DGS
- added Q1, Q10, Q12, Q13, Q14, Q16, Q3, Q4, Q6, Q7, Q9: BC817-40, Package_TO_SOT_SMD:SOT-23, symbol Device:Q_NPN_BEC
- added Q11, Q2, Q5, Q8: BC807-40, Package_TO_SOT_SMD:SOT-23, symbol Device:Q_PNP_BEC
- added Q15: IRLR3636, Package_TO_SOT_SMD:TO-252-3_TabPin2, symbol Device:Q_NMOS_GDS
Connections:
- net +15V: now also Q11.2 (E), Q2.2 (E), Q5.2 (E), Q8.2 (E)
- net BELL: now also Q15.1 (G)
- net GND: now also Q1.2 (E), Q10.2 (E), Q12.2 (E), Q13.2 (E), Q14.2 (E), Q15.3 (S), Q16.2 (E), Q3.2 (E), Q4.2 (E), Q6.2 (E), Q7.2 (E), Q9.2 (E)
- net at J2.1 (Pin_1): now also Q2.3 (C)
- net at J2.4 (Pin_4), J6.4 (Pin_4), J8.4 (Pin_4)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: now also J4.4 (Pin_4)
- net at J4.1 (Pin_1): now also Q5.3 (C)
- net at J6.1 (Pin_1): now also Q8.3 (C)
- net at J8.1 (Pin_1): now also Q11.3 (C)
- net at R6.2: now also Q3.3 (C)
- net at R4.2: now also Q3.1 (B)
- net at R13.2: now also Q6.3 (C)
- net at R11.2: now also Q6.1 (B)
- net at R18.2: now also Q9.3 (C)
- net at R16.2: now also Q9.1 (B)
- net at R22.2: now also Q12.3 (C)
- net at R21.2: now also Q12.1 (B)
- net at R24.2: now also Q13.3 (C)
- net at R23.2: now also Q13.1 (B)
- net at R26.2: now also Q14.3 (C)
- net at R25.2: now also Q14.1 (B)
- net at R31.2: now also Q16.3 (C)
- net at R28.2: now also Q16.1 (B)
- net at R2.2, R3.1: now also Q2.1 (B)
- net at R7.2, R8.1: now also Q5.1 (B)
- net at R14.2, R15.1: now also Q8.1 (B)
- net at R19.2, R20.1: now also Q11.1 (B)
- net at R3.2: now also Q1.3 (C)
- net at R1.2: now also Q1.1 (B)
- net at R8.2: now also Q4.3 (C)
- net at R5.2: now also Q4.1 (B)
- net at R15.2: now also Q7.3 (C)
- net at R12.2: now also Q7.1 (B)
- net at R20.2: now also Q10.3 (C)
- net at R17.2: now also Q10.1 (B)
- net at BZ1.2 (+), D1.2 (A): now also Q15.2 (D)

Commit message: new pcb
Parts:
- removed Q1, Q10, Q12, Q13, Q14, Q16, Q3, Q4, Q6, Q7, Q9: BC817-40, Package_TO_SOT_SMD:SOT-23, symbol Device:Q_NPN_BEC
- removed Q11, Q2, Q5, Q8: BC807-40, Package_TO_SOT_SMD:SOT-23, symbol Device:Q_PNP_BEC
- removed R1, R11, R12, R14, R16, R17, R19, R2, R21, R23, R25, R28, R4, R5, R7: 1k, Resistor_SMD:R_0603_1608Metric, symbol Device:R
- removed R13, R18, R22, R24, R26, R31, R6: 100R, Resistor_SMD:R_0603_1608Metric, symbol Device:R
- removed R15, R20, R3, R8: 10k, Resistor_SMD:R_0603_1608Metric, symbol Device:R
- added C14: 10u, Capacitor_THT:CP_Radial_D10.0mm_P5.00mm, symbol Device:C
- added C15: 100n, Capacitor_SMD:C_0603_1608Metric, symbol Device:C
- added U6: ULN2003, Package_DIP:DIP-16_W7.62mm, symbol Transistor_Array:ULN2003
- added U7: L293D, Package_DIP:DIP-16_W7.62mm, symbol Driver_Motor:L293D
Connections:
- net +12V: no longer U5.3 (VI)
- net +15V: now also U6.9 (COM), U7.8 (VCC2)
- net +24V: now also U5.3 (VI), C14.1, C15.1
- net +3V3: now also U7.1 (EN1,2), U7.16 (VCC1), U7.9 (EN3,4)
- net BELL: now also U4.25 (PA15); no longer U4.15 (PB1)
- net BUTTON_BACK: now also U4.15 (PB1); no longer U4.19 (PA9)
- net BUTTON_DOWN: now also J9.5 (Pin_5), U4.14 (PB0); no longer J9.4 (Pin_4), U4.21 (PA11)
- net BUTTON_ENTER: now also J9.3 (Pin_3), U4.12 (PA6); no longer J9.5 (Pin_5), U4.20 (PA10)
- net BUTTON_LEFT: now also U4.11 (PA5); no longer U4.23 (PA13)
- net BUTTON_RIGHT: now also J9.4 (Pin_4), U4.13 (PA7); no longer J9.3 (Pin_3), U4.22 (PA12)
- net BUTTON_UP: now also U4.10 (PA4); no longer U4.24 (PA14)
- net D1: now also U7.2 (1A)
- net D2: now also U7.7 (2A)
- net D3: now also U7.10 (3A)
- net D4: now also U7.15 (4A)
- net GND: now also C14.2, C15.2, U6.8 (GND), U7.12 (GND), U7.13 (GND), U7.4 (GND), U7.5 (GND)
- net SA: now also U4.22 (PA12), U6.3 (I3); no longer U4.26 (PB3)
- net SB: now also U4.21 (PA11), U6.4 (I4); no longer U4.25 (PA15)
- net SC: now also U4.18 (PA8), U6.7 (I7); no longer U4.13 (PA7)
- net SD: now also U4.19 (PA9), U6.6 (I6); no longer U4.12 (PA6)
- net SE: now also U4.20 (PA10), U6.5 (I5); no longer U4.11 (PA5)
- net SF: now also U4.23 (PA13), U6.2 (I2); no longer U4.27 (PB4)
- net SG: now also U4.24 (PA14), U6.1 (I1); no longer U4.28 (PB5)
- net SP: now also U4.26 (PB3); no longer U4.14 (PB0)
- net at J1.1 (Pin_1), J3.1 (Pin_1), J5.1 (Pin_1)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: now also U6.13 (O4)
- net at J1.2 (Pin_2), J3.2 (Pin_2), J5.2 (Pin_2)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: now also U6.14 (O3)
- net at J1.3 (Pin_3): now also J2.1 (Pin_1), U7.3 (1Y)
- net at J1.4 (Pin_4), J3.4 (Pin_4), J5.4 (Pin_4)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: now also U6.15 (O2)
- net at J1.5 (Pin_5), J3.5 (Pin_5), J5.5 (Pin_5)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: now also U6.16 (O1)
- net at J2.2 (Pin_2), J4.2 (Pin_2), J6.2 (Pin_2)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: now also U6.12 (O5)
- net at J2.3 (Pin_3), J4.3 (Pin_3), J6.3 (Pin_3)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: now also U6.11 (O6)
- net at J2.4 (Pin_4), J4.4 (Pin_4), J6.4 (Pin_4)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: now also U6.10 (O7)
- net at J3.3 (Pin_3): now also J4.1 (Pin_1), U7.6 (2Y)
- net at J5.3 (Pin_3): now also J6.1 (Pin_1), U7.11 (3Y)
- net at J7.3 (Pin_3): now also J8.1 (Pin_1), U7.14 (4Y)
- no-connect marks 0 -> 8
Other:
- moved on the sheet: BT1, C1, C11, C12, C13, C2, C3, C4, C5, C6, C7, C8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
