File: doc/PCB/HALL/HALL.kicad_pcb (KiCad board)
At the start: 2 copper layers, 91 parts, among them J1 Conn_01x05_Female, J10 CHIN+, J11 CHIN-, J12 Vcc, J13 CHOUT+, J14 CHOUT-, J2 Digit1, J3 Conn_01x05_Female, J4 Digit2, J5 Conn_01x05_Female, J6 Digit3, J7 Conn_01x05_Female, J8 Digit4, J9 PILOT, Q1 BC817-40, Q10 BC817-40, Q11 BC807-40, Q12 BC817-40, Q13 BC817-40, Q14 BC817-40, Q15 IRLR3636, Q16 BC817-40, Q2 BC807-40, Q3 BC817-40, Q4 BC817-40, Q5 BC807-40, Q6 BC817-40, Q7 BC817-40, Q8 BC807-40, Q9 BC817-40, SW1 UP, SW2 LEFT, SW3 RIGHT, SW4 DOWN, SW5 ENTER, SW6 BACK, U1 LM317_3PinPackage, U2 LM7812_TO220, U3 LM1117-3.3, U4 STM32F030K6Tx, U5 LM317_3PinPackage, Y1 Crystal

Commit message: PCB almost done
Parts:
- Q15: footprint Package_TO_SOT_SMD:TO-252-2 -> Package_TO_SOT_SMD:TO-252-3_TabPin2
- moved Q8 224.6 mm to (30.2, 62.8), turned to 270 degrees
- moved R8 224.1 mm to (34.0, 44.6)
- moved Q4 222.5 mm to (35.9, 48.5), turned to 180 degrees
- moved Q2 220.2 mm to (29.5, 37.2), turned to 270 degrees
- moved R19 218.3 mm to (30.5, 73.5)
- moved R17 218.1 mm to (42.1, 79.5), turned to 180 degrees
- moved R2 215.9 mm to (29.7, 32.9)
- moved R3 210.3 mm to (34.0, 32.9)
- moved Q5 210.2 mm to (29.8, 48.9), turned to 270 degrees
- moved R5 208.2 mm to (40.1, 49.5), turned to 180 degrees
- moved R14 206.8 mm to (30.4, 57.9)
- moved R7 205.1 mm to (29.9, 44.6)
- moved Q7 204.2 mm to (36.5, 62.8), turned to 180 degrees
- moved R20 201.4 mm to (35.4, 73.8)
- moved R12 199.8 mm to (41.0, 63.7), turned to 180 degrees
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Connections:
- J4 pad 4: Net-(J4-Pad4) -> Net-(J2-Pad4)
- Q1 pad 2: Net-(Q1-Pad2) -> GND
- Q1 pad 3: GND -> Net-(Q1-Pad3)
- Q10 pad 2: Net-(Q10-Pad2) -> GND
- Q10 pad 3: GND -> Net-(Q10-Pad3)
- Q11 pad 1: +15V -> Net-(Q11-Pad1)
- Q11 pad 2: Net-(J8-Pad1) -> +15V
- Q11 pad 3: Net-(Q11-Pad3) -> Net-(J8-Pad1)
- Q12 pad 2: Net-(Q12-Pad2) -> GND
- Q12 pad 3: GND -> Net-(Q12-Pad3)
- Q13 pad 2: Net-(Q13-Pad2) -> GND
- Q13 pad 3: GND -> Net-(Q13-Pad3)
- Q14 pad 2: Net-(Q14-Pad2) -> GND
- Q14 pad 3: GND -> Net-(Q14-Pad3)
- Q15 pad 1: Net-(BZ1-Pad2) -> BELL
- Q15 pad 2: BELL -> Net-(BZ1-Pad2)
- Q16 pad 2: Net-(Q16-Pad2) -> GND
- Q16 pad 3: GND -> Net-(Q16-Pad3)
- Q2 pad 1: +15V -> Net-(Q2-Pad1)
- Q2 pad 2: Net-(J2-Pad1) -> +15V
- Q2 pad 3: Net-(Q2-Pad3) -> Net-(J2-Pad1)
- Q3 pad 2: Net-(Q3-Pad2) -> GND
- Q3 pad 3: GND -> Net-(Q3-Pad3)
- Q4 pad 2: Net-(Q4-Pad2) -> GND
- Q4 pad 3: GND -> Net-(Q4-Pad3)
- Q5 pad 1: +15V -> Net-(Q5-Pad1)
- Q5 pad 2: Net-(J4-Pad1) -> +15V
- Q5 pad 3: Net-(Q5-Pad3) -> Net-(J4-Pad1)
- Q6 pad 2: Net-(Q6-Pad2) -> GND
- Q6 pad 3: GND -> Net-(Q6-Pad3)
- Q7 pad 2: Net-(Q7-Pad2) -> GND
- Q7 pad 3: GND -> Net-(Q7-Pad3)
- Q8 pad 1: +15V -> Net-(Q8-Pad1)
- Q8 pad 2: Net-(J6-Pad1) -> +15V
- Q8 pad 3: Net-(Q8-Pad3) -> Net-(J6-Pad1)
- Q9 pad 2: Net-(Q9-Pad2) -> GND
- Q9 pad 3: GND -> Net-(Q9-Pad3)
- R1 pad 2: Net-(Q1-Pad2) -> Net-(Q1-Pad1)
- R11 pad 2: Net-(Q6-Pad2) -> Net-(Q6-Pad1)
- R12 pad 2: Net-(Q7-Pad2) -> Net-(Q7-Pad1)
- R13 pad 2: Net-(Q6-Pad1) -> Net-(Q6-Pad3)
- R14 pad 2: Net-(Q8-Pad3) -> Net-(Q8-Pad1)
- R15 pad 1: Net-(Q8-Pad3) -> Net-(Q8-Pad1)
- R15 pad 2: Net-(Q7-Pad1) -> Net-(Q7-Pad3)
- R16 pad 2: Net-(Q9-Pad2) -> Net-(Q9-Pad1)
- R17 pad 2: Net-(Q10-Pad2) -> Net-(Q10-Pad1)
- R18 pad 2: Net-(Q9-Pad1) -> Net-(Q9-Pad3)
- R19 pad 2: Net-(Q11-Pad3) -> Net-(Q11-Pad1)
- R2 pad 2: Net-(Q2-Pad3) -> Net-(Q2-Pad1)
- R20 pad 1: Net-(Q11-Pad3) -> Net-(Q11-Pad1)
- R20 pad 2: Net-(Q10-Pad1) -> Net-(Q10-Pad3)
- R21 pad 2: Net-(Q12-Pad2) -> Net-(Q12-Pad1)
- R22 pad 2: Net-(Q12-Pad1) -> Net-(Q12-Pad3)
- R23 pad 2: Net-(Q13-Pad2) -> Net-(Q13-Pad1)
- R24 pad 2: Net-(Q13-Pad1) -> Net-(Q13-Pad3)
- R25 pad 2: Net-(Q14-Pad2) -> Net-(Q14-Pad1)
- R26 pad 2: Net-(Q14-Pad1) -> Net-(Q14-Pad3)
- R28 pad 2: Net-(Q16-Pad2) -> Net-(Q16-Pad1)
- R3 pad 1: Net-(Q2-Pad3) -> Net-(Q2-Pad1)
- R3 pad 2: Net-(Q1-Pad1) -> Net-(Q1-Pad3)
- R31 pad 2: Net-(Q16-Pad1) -> Net-(Q16-Pad3)
- R4 pad 2: Net-(Q3-Pad2) -> Net-(Q3-Pad1)
- R5 pad 2: Net-(Q4-Pad2) -> Net-(Q4-Pad1)
- R6 pad 2: Net-(Q3-Pad1) -> Net-(Q3-Pad3)
- R7 pad 2: Net-(Q5-Pad3) -> Net-(Q5-Pad1)
- R8 pad 1: Net-(Q5-Pad3) -> Net-(Q5-Pad1)
- R8 pad 2: Net-(Q4-Pad1) -> Net-(Q4-Pad3)
Routing:
- net Net-(J1-Pad1): track 0.00 -> 142.6 mm, vias 0 -> 1
- net Net-(J2-Pad4): track 0.00 -> 139.7 mm
- net Net-(J1-Pad2): track 0.00 -> 133.0 mm, vias 0 -> 1
- net Net-(J8-Pad1): track 0.00 -> 128.4 mm, vias 0 -> 1
- net Net-(J2-Pad3): track 0.00 -> 128.1 mm
- net Net-(J1-Pad4): track 0.00 -> 127.0 mm
- net Net-(J2-Pad2): track 0.00 -> 121.7 mm
- net Net-(J1-Pad5): track 0.00 -> 118.0 mm, vias 0 -> 1
- net SC: track 0.00 -> 117.1 mm, vias 0 -> 2
- net SB: track 0.00 -> 111.0 mm, vias 0 -> 2
- net SA: track 0.00 -> 102.2 mm, vias 0 -> 2
- net SD: track 0.00 -> 101.5 mm, vias 0 -> 2
- net Net-(J6-Pad1): track 0.00 -> 94.3 mm, vias 0 -> 1
- net SF: track 0.00 -> 91.7 mm, vias 0 -> 2
- net SE: track 0.00 -> 90.8 mm, vias 0 -> 2
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- added copper zone on B.Cu, net GND
Other:
- board outline added: 161.7 x 105.8 mm

Commit message: new pcb
Parts:
- removed Q1, Q10, Q12, Q13, Q14, Q16, Q3, Q4, Q6, Q7, Q9: BC817-40, Package_TO_SOT_SMD:SOT-23
- removed Q11, Q2, Q5, Q8: BC807-40, Package_TO_SOT_SMD:SOT-23
- removed R1, R11, R12, R14, R16, R17, R19, R2, R21, R23, R25, R28, R4, R5, R7: 1k, Resistor_SMD:R_0603_1608Metric
- removed R13, R18, R22, R24, R26, R31, R6: 100R, Resistor_SMD:R_0603_1608Metric
- removed R15, R20, R3, R8: 10k, Resistor_SMD:R_0603_1608Metric
- removed SW1: UP, Button_Switch_SMD:SW_SPST_CK_RS282G05A3
- removed SW2: LEFT, Button_Switch_SMD:SW_SPST_CK_RS282G05A3
- removed SW3: RIGHT, Button_Switch_SMD:SW_SPST_CK_RS282G05A3
- removed SW4: DOWN, Button_Switch_SMD:SW_SPST_CK_RS282G05A3
- removed SW5: ENTER, Button_Switch_SMD:SW_SPST_CK_RS282G05A3
- removed SW6: BACK, Button_Switch_SMD:SW_SPST_CK_RS282G05A3
- added C14: 10u, Capacitor_THT:CP_Radial_D10.0mm_P5.00mm, F.Cu at (39.8, 83.0)
- added C15: 100n, Capacitor_SMD:C_0603_1608Metric, F.Cu at (48.5, 83.8)
- added U6: ULN2003, Package_DIP:DIP-16_W7.62mm, F.Cu at (92.6, 49.9)
- added U7: L293D, Package_DIP:DIP-16_W7.62mm, F.Cu at (46.2, 18.4)
- moved J9 87.2 mm to (63.3, 99.4), turned to 90 degrees
- moved C8 70.3 mm to (147.4, 68.5), turned to 180 degrees
- moved BZ1 57.4 mm to (135.6, 40.6), turned to 0 degrees
- moved Q15 55.3 mm to (133.4, 53.4), turned to 0 degrees
- moved U2 51.6 mm to (95.3, 73.2), turned to 90 degrees
- moved D1 49.7 mm to (128.8, 40.6), turned to 270 degrees
- moved C11 46.0 mm to (112.2, 68.1), turned to 270 degrees
- moved C12 45.7 mm to (119.0, 66.0)
- moved U3 43.7 mm to (145.7, 89.2), turned to 0 degrees
- moved R27 38.7 mm to (123.0, 54.9), turned to 270 degrees
- moved J12 36.1 mm to (34.5, 61.0)
- moved C13 34.7 mm to (70.9, 86.4), turned to 270 degrees
- moved U5 32.7 mm to (61.2, 88.1), turned to 90 degrees
- moved C2 28.3 mm to (48.8, 70.0)
- moved R9 27.0 mm to (66.5, 74.3), turned to 270 degrees
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Connections:
- J2 pad 1: Net-(J2-Pad1) -> Net-(J1-Pad3)
- J4 pad 1: Net-(J4-Pad1) -> Net-(J3-Pad3)
- J6 pad 1: Net-(J6-Pad1) -> Net-(J5-Pad3)
- J8 pad 1: Net-(J8-Pad1) -> Net-(J7-Pad3)
- J9 pad 3: BUTTON_RIGHT -> BUTTON_ENTER
- J9 pad 4: BUTTON_DOWN -> BUTTON_RIGHT
- J9 pad 5: BUTTON_ENTER -> BUTTON_DOWN
- U4 pad 10: Net-(U4-Pad10) -> BUTTON_UP
- U4 pad 11: SE -> BUTTON_LEFT
- U4 pad 12: SD -> BUTTON_ENTER
- U4 pad 13: SC -> BUTTON_RIGHT
- U4 pad 14: SP -> BUTTON_DOWN
- U4 pad 15: BELL -> BUTTON_BACK
- U4 pad 18: Net-(U4-Pad18) -> SC
- U4 pad 19: BUTTON_BACK -> SD
- U4 pad 20: BUTTON_ENTER -> SE
- U4 pad 21: BUTTON_DOWN -> SB
- U4 pad 22: BUTTON_RIGHT -> SA
- U4 pad 23: BUTTON_LEFT -> SF
- U4 pad 24: BUTTON_UP -> SG
- U4 pad 25: SB -> BELL
- U4 pad 26: SA -> SP
- U4 pad 27: SF -> Net-(U4-Pad27)
- U4 pad 28: SG -> Net-(U4-Pad28)
- U5 pad 3: +12V -> +24V
Routing:
- net Net-(J8-Pad1): track 128.4 -> 0.00 mm, vias 1 -> 0
- net Net-(J7-Pad3): track 0.00 -> 102.2 mm, vias 0 -> 1
- net Net-(J6-Pad1): track 94.3 -> 0.00 mm, vias 1 -> 0
- net Net-(J5-Pad3): track 0.00 -> 89.8 mm, vias 0 -> 2
- net SB: track 111.0 -> 27.2 mm, vias 2 -> 0
- net SC: track 117.1 -> 35.8 mm, vias 2 -> 0
- net Net-(J3-Pad3): track 0.00 -> 81.0 mm
- net SA: track 102.2 -> 24.3 mm, vias 2 -> 0
- net SF: track 91.7 -> 21.5 mm, vias 2 -> 0
- net SD: track 101.5 -> 33.2 mm, vias 2 -> 0
- net SG: track 81.5 -> 19.3 mm, vias 2 -> 0
- net SE: track 90.8 -> 30.1 mm, vias 2 -> 0
- net Net-(J4-Pad1): track 59.1 -> 0.00 mm, vias 1 -> 0
- net +24V: track 33.6 -> 89.3 mm
- net +3V3: track 114.4 -> 168.8 mm
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Other:
- board size 161.7 x 105.8 mm -> 120 x 90.2 mm

Commit message: new pcb
Routing:
- net D4: track 69.3 -> 67.6 mm
- net GND: vias 0 -> 2
Changed lines of the file:
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@@
     (thickness 1.6)
     (drawings 8)
-    (tracks 418)
+    (tracks 422)
     (zones 0)
     (modules 48)
@@
   )
   (setup
-    (last_trace_width 1)
+    (last_trace_width 0.4)
     (user_trace_width 0.4)
     (user_trace_width 1)
@@
   (segment (start 53.87 26.02) (end 53.87 28.56) (width 0.4) (layer F.Cu) (net 2))
   (segment (start 46.25 26.02) (end 46.25 28.56) (width 0.4) (layer F.Cu) (net 2))
+  (via (at 42.06 28.61) (size 2) (drill 0.8) (layers F.Cu B.Cu) (net 2))
+  (via (at 54.48 43.8) (size 2) (drill 0.8) (layers F.Cu B.Cu) (net 2))
   (segment (start 61.2 85.56) (end 64.64 85.56) (width 2) (layer F.Cu) (net 3))
   (segment (start 64.64 85.56) (end 67.25 82.95) (width 2) (layer F.Cu) (net 3))
@@
   (segment (start 49.602916 61.4) (end 46.75 58.547084) (width 0.4) (layer F.Cu) (net 40))
   (segment (start 64.375 61.4) (end 49.602916 61.4) (width 0.4) (layer F.Cu) (net 40))
-  (via (at 45.5 43) (size 2) (drill 0.8) (layers F.Cu B.Cu) (net 40))
-  (segment (start 46.75 58.547084) (end 46.75 44.25) (width 0.4) (layer F.Cu) (net 40))
-  (segment (start 46.75 44.25) (end 45.5 43) (width 0.4) (layer F.Cu) (net 40))
+  (via (at 45.36 48.22) (size 2) (drill 0.8) (layers F.Cu B.Cu) (net 40))
   (segment (start 46.499999 41.010001) (end 53.070001 34.439999) (width 0.4) (layer B.Cu) (net 40))
-  (segment (start 46.499999 42.000001) (end 46.499999 41.010001) (width 0.4) (layer B.Cu) (net 40))
   (segment (start 53.070001 34.439999) (end 53.87 33.64) (width 0.4) (layer B.Cu) (net 40))
-  (segment (start 45.5 43) (end 46.499999 42.000001) (width 0.4) (layer B.Cu) (net 40))
-  (via (at 43.55 40.15) (size 2) (drill 0.8) (layers F.Cu B.Cu) (net 41))
-  (segment (start 43.55 56.195626) (end 43.55 40.15) (width 0.4) (layer F.Cu) (net 41))
+  (segment (start 46.499999 42.000001) (end 46.499999 41.010001) (width 0.4) (layer B.Cu) (net 40))
+  (segment (start 45.36 43.14) (end 46.499999 42.000001) (width 0.4) (layer B.Cu) (net 40))
+  (segment (start 45.36 48.22) (end 45.36 43.14) (width 0.4) (layer B.Cu) (net 40))
+  (segment (start 46.75 49.61) (end 45.36 48.22) (width 0.4) (layer F.Cu) (net 40))
+  (segment (start 46.75 58.547084) (end 46.75 49.61) (width 0.4) (layer F.Cu) (net 40))
+  (via (at 43.61 45.59) (size 2) (drill 0.8) (layers F.Cu B.Cu) (net 41))
   (segment (start 49.354383 62.000009) (end 43.55 56.195626) (width 0.4) (layer F.Cu) (net 41))
   (segment (start 68.4 60.125) (end 66.524991 62.000009) (width 0.4) (layer F.Cu) (net 41))
   (segment (start 66.524991 62.000009) (end 49.354383 62.000009) (width 0.4) (layer F.Cu) (net 41))
-  (segment (start 43.55 40.15) (end 46.511458 40.15) (width 0.4) (layer B.Cu) (net 41))
-  (segment (start 46.511458 40.15) (end 50.95 35.711458) (width 0.4) (layer B.Cu) (net 41))
-  (segment (start 50.95 23.86) (end 53.87 20.94) (width 0.4) (layer B.Cu) (net 41))
-  (segment (start 50.95 35.711458) (end 50.95 23.86) (width 0.4) (layer B.Cu) (net 41))
+  (segment (start 43.61 43.051458) (end 43.61 45.59) (width 0.4) (layer B.Cu) (net 41))
+  (segment (start 50.95 35.711458) (end 43.61 43.051458) (width 0.4) (layer B.Cu) (net 41))
+  (segment (start 53.87 20.94) (end 50.95 23.86) (width 0.4) (layer B.Cu) (net 41))
+  (segment (start 50.95 23.86) (end 50.95 35.711458) (width 0.4) (layer B.Cu) (net 41))
+  (segment (start 43.61 56.135626) (end 43.61 45.59) (width 0.4) (layer F.Cu) (net 41))
+  (segment (start 43.55 56.195626) (end 43.61 56.135626) (width 0.4) (layer F.Cu) (net 41))
   (segment (start 96.26 56.35) (end 102.76 49.85) (width 0.4) (layer F.Cu) (net 42))
   (segment (start 75.375 56.35) (end 96.26 56.35) (width 0.4) (layer F.Cu) (net 42))
